Commit message: 0412jianmo

File: src/robot_description/urdf/diff_drive_base.xacro (robot description, xacro)
@@ -88,10 +88,9 @@
       <parent link="base_link"/>
       <child  link="${prefix}_wheel_link"/>
-      <!-- 轮心离地面高度 = wheel_radius
-           相对 base_link 中心 Z = wheel_radius - chassis_z_offset -->
-      <origin xyz="${wheel_x_offset}
-                   ${y_sign * wheel_y_offset}
-                   ${wheel_radius - chassis_z_offset}"
-              rpy="0 0 0"/>
+      <!-- 轮心相对 base_link 中心:
+           x = wheel_x_offset (0)
+           y = ±wheel_y_offset (轮距/2)
+           z = wheel_radius - chassis_z_offset (轮心在底盘中心下方) -->
+      <origin xyz="${wheel_x_offset} ${y_sign * wheel_y_offset} ${wheel_radius - chassis_z_offset}" rpy="0 0 0"/>
       <!-- 旋转轴: Y轴 -->
       <axis xyz="0 1 0"/>
@@ -127,5 +126,5 @@
        ===================================== -->
   <xacro:macro name="caster_wheel" params="prefix x_pos y_pos">
-    <link name="${prefix}_caster_link">
+    <link name="${prefix}_link">
       <visual>
         <origin xyz="0 0 0" rpy="0 0 0"/>
@@ -143,12 +142,15 @@
       <xacro:sphere_inertia m="${caster_mass}" r="${caster_radius}"/>
     </link>
-    <joint name="${prefix}_caster_joint" type="fixed">
+    <joint name="${prefix}_joint" type="fixed">
       <parent link="base_link"/>
-      <child  link="${prefix}_caster_link"/>
-      <!-- Z: 底盘底面 - 脚轮半径 = 脚轮球心高度 -->
-      <origin xyz="${x_pos} ${y_pos} ${-chassis_height/2 - caster_radius}" rpy="0 0 0"/>
+      <child  link="${prefix}_link"/>
+      <!-- 脚轮球心接地时高度 = caster_radius
+           相对 base_link 中心 z = caster_radius - chassis_z_offset
+           与驱动轮同理: wheel_radius - chassis_z_offset
+           D1: 0.0127 - 0.14275 = -0.13005m -->
+      <origin xyz="${x_pos} ${y_pos} ${caster_radius - chassis_z_offset}" rpy="0 0 0"/>
     </joint>
     <!-- 脚轮设置低摩擦, 允许自由滑动 -->
-    <gazebo reference="${prefix}_caster_link">
+    <gazebo reference="${prefix}_link">
       <mu1>0.0</mu1>
       <mu2>0.0</mu2>
@@ -163,3 +165,70 @@
                       x_pos="${caster_x_rear}"
                       y_pos="0.0"/>
+  <!-- =====================================================
+       上层平台: 4 根支撑柱 + 顶部圆盘
+       与实物 EAI D1 对应:
+         4根细圆柱从底盘顶面延伸, 承托上层圆盘
+         上层圆盘与底盘同半径, 厚 8mm
+       ===================================================== -->
+  <!-- 支撑柱宏: prefix=FL/FR/RL/RR, x_sign=±1, y_sign=±1 -->
+  <xacro:macro name="support_pillar" params="prefix x_sign y_sign">
+    <link name="pillar_${prefix}_link">
+      <visual>
+        <origin xyz="0 0 0" rpy="0 0 0"/>
+        <geometry>
+          <cylinder radius="${pillar_radius}" length="${pillar_height}"/>
+        </geometry>
+        <material name="dark_gray"/>
+      </visual>
+      <collision>
+        <origin xyz="0 0 0" rpy="0 0 0"/>
+        <geometry>
+          <cylinder radius="${pillar_radius}" length="${pillar_height}"/>
+        </geometry>
+      </collision>
+      <xacro:cylinder_inertia m="${pillar_mass}" r="${pillar_radius}" h="${pillar_height}"/>
+    </link>
+    <joint name="pillar_${prefix}_joint" type="fixed">
+      <parent link="base_link"/>
+      <child  link="pillar_${prefix}_link"/>
+      <!-- 柱子中心: 底盘顶面 + 柱子半高
+           z = chassis_height/2 + pillar_height/2 -->
+      <origin xyz="${x_sign * pillar_xy_offset} ${y_sign * pillar_xy_offset} ${chassis_height/2 + pillar_height/2}" rpy="0 0 0"/>
+    </joint>
+    <gazebo reference="pillar_${prefix}_link">
+      <material>Gazebo/DarkGrey</material>
+    </gazebo>
+  </xacro:macro>
+  <!-- 四角支撑柱 (前左/前右/后左/后右) -->
+  <xacro:support_pillar prefix="FL" x_sign="1"  y_sign="1"/>
+  <xacro:support_pillar prefix="FR" x_sign="1"  y_sign="-1"/>
+  <xacro:support_pillar prefix="RL" x_sign="-1" y_sign="1"/>
+  <xacro:support_pillar prefix="RR" x_sign="-1" y_sign="-1"/>
+  <!-- 顶部圆盘平台 -->
+  <link name="top_plate_link">
+    <visual>
+      <origin xyz="0 0 0" rpy="0 0 0"/>
+      <geometry>
+        <cylinder radius="${top_plate_radius}" length="${top_plate_height}"/>
+      </geometry>
+      <material name="dark_gray"/>
+    </visual>
+    <collision>
+      <origin xyz="0 0 0" rpy="0 0 0"/>
+      <geometry>
+        <cylinder radius="${top_plate_radius}" length="${top_plate_height}"/>
+      </geometry>
+    </collision>
+    <xacro:cylinder_inertia m="${top_plate_mass}" r="${top_plate_radius}" h="${top_plate_height}"/>
+  </link>
+  <joint name="top_plate_joint" type="fixed">
+    <parent link="base_link"/>
+    <child  link="top_plate_link"/>
+    <!-- 顶盘中心: 底盘顶面 + 柱子高度 + 顶盘半厚
+         z = chassis_height/2 + pillar_height + top_plate_height/2 -->
+    <origin xyz="0 0 ${chassis_height/2 + pillar_height + top_plate_height/2}" rpy="0 0 0"/>
+  </joint>
+  <gazebo reference="top_plate_link">
+    <material>Gazebo/DarkGrey</material>
+  </gazebo>
 </robot>

File: src/robot_description/urdf/gazebo_control.xacro (robot description, xacro)
@@ -26,9 +26,8 @@
       <left_joint>left_wheel_joint</left_joint>
       <right_joint>right_wheel_joint</right_joint>
-      <!-- 轮子半径(m) 与 robot_params.xacro 中 wheel_radius 一致 -->
-      <wheel_radius>0.0508</wheel_radius>
-      <!-- 轮距(m): D1文档实测值 0.3559m -->
-      <wheel_separation>0.3559</wheel_separation>
-      <!-- 最大线速度(m/s) 【TODO】根据电机最大转速和轮径计算 -->
+      <!-- 轮子直径(m): Φ125mm = 0.125m -->
+      <wheel_diameter>0.125</wheel_diameter>
+      <!-- 轮距(m): 图纸标注 350.7mm -->
+      <wheel_separation>0.3507</wheel_separation>      <!-- 最大线速度(m/s) 【TODO】根据电机最大转速和轮径计算 -->
       <max_wheel_torque>20.0</max_wheel_torque>
       <!-- 最大角加速度(rad/s^2) -->

File: src/robot_description/urdf/robot_params.xacro (robot description, xacro)
@@ -16,14 +16,14 @@
   <xacro:property name="chassis_mass"     value="20.0"/>
   <!-- =================== 驱动轮参数 ===================
-       D1 实测参数:
-         wheel_radius   : 4寸橡胶轮半径 4x25.4/2 = 0.0508m
+       D1 图纸实测参数:
+         wheel_radius   : 驱动轮 Φ125mm → 半径 0.0625m
          wheel_width    : 轮宽 ~0.04m (待实测)
          wheel_mass     : 单轮质量估算 ~1.0kg
-         wheel_y_offset : 轮距/2 = 0.3559/2 = 0.17795m
+         wheel_y_offset : 轮距/2 = 350.7mm/2 = 0.17535m
   -->
-  <xacro:property name="wheel_radius"     value="0.0508"/>
+  <xacro:property name="wheel_radius"     value="0.0625"/>
   <xacro:property name="wheel_width"      value="0.04"/>
   <xacro:property name="wheel_mass"       value="1.0"/>
-  <xacro:property name="wheel_y_offset"   value="0.17795"/>
+  <xacro:property name="wheel_y_offset"   value="0.17535"/>
   <xacro:property name="wheel_x_offset"   value="0.0"/>
   <!-- =================== 万向支撑轮参数 ===================
@@ -44,26 +44,42 @@
   -->
   <xacro:property name="chassis_z_offset" value="${0.038 + chassis_height/2}"/>
+  <!-- =================== 上层圆盘平台参数 ===================
+       4根柱子支撑上层圆盘, 外观参考实物图:
+         pillar_height   : 柱子高度 ≈ chassis_height * 0.6
+         pillar_radius   : 细圆柱半径
+         pillar_xy_offset: 柱子分布在圆盘半径70%处
+         top_plate_radius: 上层圆盘半径 = chassis_radius
+         top_plate_height: 上层圆盘厚度
+  -->
+  <xacro:property name="pillar_height"     value="${chassis_height * 0.6}"/>
+  <xacro:property name="pillar_radius"     value="0.015"/>
+  <xacro:property name="pillar_mass"       value="0.5"/>
+  <xacro:property name="pillar_xy_offset"  value="${chassis_radius * 0.7}"/>
+  <xacro:property name="top_plate_radius"  value="${chassis_radius}"/>
+  <xacro:property name="top_plate_height"  value="0.008"/>
+  <xacro:property name="top_plate_mass"    value="1.0"/>
   <!-- =================== 3D激光雷达安装参数 ===================
-       前置安装在底盘顶面前沿 (x ≈ chassis_radius*0.8):
-         lidar_x = 0.16m (圆形底盘前沿内侧)
-         lidar_y = 0.0   (居中)
-         lidar_z = chassis_height/2 + 支架0.05m + 雷达半高0.03m
-       【TODO】雷达型号确定后校对 lidar_radius/lidar_height
+       雷达位置由外参标定 + 相机已知位置反推:
+         相机已知(top_plate坐标系): x=0.15, y=0.0, z=0.019
+         雷达位置 = 相机位置 - R_pitch(-28.3°) × t
+         结果: lidar_x=-0.006m, lidar_y=-0.037m, z=0.027m
+         即雷达在相机后方偏右、几乎等高，与实物图吹合
+       rpy pitch=-0.4947 rad (-28.3°): 由外参矩阵第3列反推
   -->
-  <xacro:property name="lidar_x"          value="0.16"/>
+  <xacro:property name="lidar_x"          value="0.10"/>
   <xacro:property name="lidar_y"          value="0.0"/>
-  <xacro:property name="lidar_z"          value="${chassis_height/2 + 0.08}"/>
+  <!-- lidar_z 已废弃, 由 sensors.xacro 中 joint origin 直接计算 -->
   <xacro:property name="lidar_mass"       value="0.83"/>
   <xacro:property name="lidar_radius"     value="0.04"/>
   <xacro:property name="lidar_height"     value="0.06"/>
   <!-- =================== 深度相机安装参数 ===================
-       前置安装, 与激光雷达同一X位置, 雷达上方:
-         camera_x = lidar_x = 0.16m
-         camera_z = chassis_height/2 + 0.18m (雷达上方约0.1m)
+       安装在上层圆盘前沿:
+         camera_x = 0.15m (圆盘前沿内侧)
+         camera_y = 0.0   (居中)
+       camera z/高度由 sensors.xacro 中 camera_joint 计算
        【TODO】相机安装高度以实际支架为准
   -->
-  <xacro:property name="camera_x"         value="0.16"/>
+  <xacro:property name="camera_x"         value="0.15"/>
   <xacro:property name="camera_y"         value="0.0"/>
-  <xacro:property name="camera_z"         value="${chassis_height/2 + 0.18}"/>
   <xacro:property name="camera_mass"      value="0.15"/>
   <xacro:property name="camera_size_x"    value="0.03"/>

File: src/robot_description/urdf/sensors.xacro (robot description, xacro)
@@ -12,31 +12,7 @@
 <robot xmlns:xacro="http://www.ros.org/wiki/xacro">
   <!-- ============================================================
-       3D激光雷达
+       3D激光雷达 (半球形)
+       与深度相机并排安装在上层圆盘前沿, 朝上覆盖半球视野
        ============================================================ -->
-  <!-- 雷达支架link -->
-  <link name="lidar_mount_link">
-    <visual>
-      <origin xyz="0 0 0" rpy="0 0 0"/>
-      <geometry>
-        <!-- 【TODO】根据实际支架尺寸调整 -->
-        <cylinder radius="0.02" length="0.08"/>
-      </geometry>
-      <material name="dark_gray"/>
-    </visual>
-    <collision>
-      <origin xyz="0 0 0" rpy="0 0 0"/>
-      <geometry>
-        <cylinder radius="0.02" length="0.08"/>
-      </geometry>
-    </collision>
-    <xacro:cylinder_inertia m="0.05" r="0.02" h="0.08"/>
-  </link>
-  <joint name="lidar_mount_joint" type="fixed">
-    <parent link="base_link"/>
-    <child  link="lidar_mount_link"/>
-    <!-- 支架安装在底盘前部顶面
-         【TODO】x/y偏移根据实际安装调整 -->
-    <origin xyz="${lidar_x} ${lidar_y} ${chassis_height/2 + 0.04}" rpy="0 0 0"/>
-  </joint>
   <!-- 雷达主体link -->
   <link name="lidar_link">
@@ -56,9 +32,15 @@
     <xacro:cylinder_inertia m="${lidar_mass}" r="${lidar_radius}" h="${lidar_height}"/>
   </link>
+  <!-- lidar_link 挂载在 top_plate_link
+       位置由外参标定矩阵反推(锁定相机位置, 推算雷达位置):
+         相机已知(top_plate): x=0.15, y=0.0, z=0.019
+         雷达位置 = 相机位置 - R_pitch(-28.3°) * t
+         结果: x=-0.006m, y=-0.037m, z=0.027m
+         即雷达在相机后方偏右，与相机几乎等高 (与实物吕合)
+       rpy pitch=-0.4947 rad (-28.3°): 由外参矩阵第3列反推 -->
   <joint name="lidar_joint" type="fixed">
-    <parent link="lidar_mount_link"/>
+    <parent link="top_plate_link"/>
     <child  link="lidar_link"/>
-    <!-- Z偏移 = 支架高度/2 + 雷达高度/2 -->
-    <origin xyz="0 0 ${0.04 + lidar_height/2}" rpy="0 0 0"/>
+    <origin xyz="${lidar_x} ${lidar_y} ${top_plate_height/2 + lidar_height/2 + 0.008}" rpy="0 -0.4947 0"/>
   </joint>
   <!-- Gazebo 3D激光雷达传感器插件 -->
@@ -74,12 +56,11 @@
       <ray>
         <scan>
-          <!-- 水平扫描: 360度, 采样点数
-               VLP-16: 1800点(0.2°分辨率) / HDL-32: 2160点
-               【TODO】horizontal_samples根据型号调整 -->
+          <!-- 水平扫描: 前180度(-90°~+90°), 采样点数
+               VLP-16: 900点(0.2°分辨率) / 只保留前半圆数据 -->
           <horizontal>
-            <samples>1800</samples>
+            <samples>900</samples>
             <resolution>1</resolution>
-            <min_angle>-3.14159265</min_angle>
-            <max_angle>3.14159265</max_angle>
+            <min_angle>-1.5707963268</min_angle>
+            <max_angle>1.5707963268</max_angle>
           </horizontal>
           <!-- 垂直扫描(线束)
@@ -130,32 +111,9 @@
   <!-- ============================================================
        深度相机 (RGB-D)
-       支持 RealSense D435/D455 风格的配置
+       挂载在 lidar_link 下方, 位置由外参标定矩阵确定:
+         T_camera_in_lidar 平移量 t = [0.1336, 0.0369, -0.0807] m
+         相机在雷达前方 13.4cm, 左方 3.7cm, 下方 8.1cm
        ============================================================ -->
-  <!-- 相机支架link -->
-  <link name="camera_mount_link">
-    <visual>
-      <origin xyz="0 0 0" rpy="0 0 0"/>
-      <geometry>
-        <!-- 【TODO】根据实际支架尺寸调整 -->
-        <box size="0.02 0.04 0.15"/>
-      </geometry>
-      <material name="dark_gray"/>
-    </visual>
-    <collision>
-      <origin xyz="0 0 0" rpy="0 0 0"/>
-      <geometry>
-        <box size="0.02 0.04 0.15"/>
-      </geometry>
-    </collision>
-    <xacro:box_inertia m="0.05" dx="0.02" dy="0.04" dz="0.15"/>
-  </link>
-  <joint name="camera_mount_joint" type="fixed">
-    <parent link="base_link"/>
-    <child  link="camera_mount_link"/>
-    <!-- 相机支架安装在底盘前部
-         【TODO】x/y偏移和z高度根据实际安装调整 -->
-    <origin xyz="${camera_x - 0.01} ${camera_y} ${chassis_height/2 + 0.075}" rpy="0 0 0"/>
-  </joint>
-  <!-- 相机主体link (RGB部分中心为光学原点) -->
+  <!-- 相机主体link -->
   <link name="camera_link">
     <visual>
@@ -177,10 +135,13 @@
                        dz="${camera_size_z}"/>
   </link>
+  <!-- 相机安装关节:
+       父节点 = top_plate_link (物理安装位置已知)
+       x=camera_x=0.15m (顶盘前沿), y=0, z=顶盘半厚+相机半高
+       rpy=0: 水平朝前
+       外参标定的旋转部分 RPY=(-1.076,0.017,-1.570) 仅用于 FAST-LIO2 算法配置 -->
   <joint name="camera_joint" type="fixed">
-    <parent link="camera_mount_link"/>
+    <parent link="top_plate_link"/>
     <child  link="camera_link"/>
-    <!-- 相机固定在支架顶部
-         【TODO】根据实际相机安装高度和水平位置调整 -->
-    <origin xyz="${camera_size_x/2} 0 ${0.075}" rpy="0 0 0"/>
+    <origin xyz="${camera_x} ${camera_y} ${top_plate_height/2 + camera_size_z/2}" rpy="0 0 0"/>
   </joint>
   <!-- ROS标准: 相机光学坐标系
